File: ALU/Hol-1-ALU.sch (KiCad schematic (older format))
At the start: 29 parts, among them P1 REGISTER A LINK, P2 REGISTER B LINK, P3 STATUS & CTRL, P4 DATA BUS, P5 DATA BUS, P6 DATA BUS, P7 DATA BUS, P8 Power, U1 74LS283, U2 74LS283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

Commit message: v1.2.2 resistor values added to schematic
Parts:
- R1: value R -> 47kΩ
- RA1: value R-ARRAY-8 -> 220Ω
Changed lines of the file:
@@
 Sheet 1 1
 Title "Hol-1 8-bit CPU - ALU board"
-Date "14 mar 2019"
+Date "16 mar 2019"
 Rev "1.0"
 Comp "www.Benningtons.Net"
@@
 P 3000 6900
 F 0 "RA1" V 3175 6925 70  0000 C CNN
-F 1 "R-ARRAY-8" V 3030 6900 70  0000 C CNN
+F 1 "220Ω" V 3030 6900 70  0000 C CNN
 F 2 "~" H 3000 6900 60  0000 C CNN
 F 3 "~" H 3000 6900 60  0000 C CNN
@@
 U 1 1 5C81D24A
 P 2475 6750
-F 0 "R1" V 2375 6750 40  0000 C CNN
-F 1 "R" V 2375 6750 40  0001 C CNN
+F 0 "R1" V 2400 6650 40  0000 C CNN
+F 1 "47kΩ" V 2400 6850 40  0000 C CNN
 F 2 "~" V 2405 6750 30  0000 C CNN
 F 3 "~" H 2475 6750 30  0000 C CNN

Commit message: v1.5.15 ALU: Re-numbered 8 pin IDC ports to reflect the anti-clockwise numbering used
Connections:
- wire segments 173 -> 186
Other:
- moved on the sheet: JP1, P2
Changed lines of the file:
@@
 Sheet 1 1
 Title "Hol-1 8-bit CPU - ALU board"
-Date "16 mar 2019"
+Date "19 jan 2020"
 Rev "1.0"
 Comp "www.Benningtons.Net"
@@
 L CONN_8 P2
 U 1 1 5C5A0CA2
-P 700 5250
-F 0 "P2" V 650 5250 60  0000 C CNN
-F 1 "REGISTER B LINK" V 750 5250 60  0000 C CNN
-F 2 "" H 700 5250 60  0000 C CNN
-F 3 "" H 700 5250 60  0000 C CNN
-	1    700  5250
-	-1   0    0    -1
+P 925 4400
+F 0 "P2" V 875 4400 60  0000 C CNN
+F 1 "REGISTER B LINK" V 975 4400 60  0000 C CNN
+F 2 "" H 925 4400 60  0000 C CNN
+F 3 "" H 925 4400 60  0000 C CNN
+	1    925  4400
+	0    1    -1   0
 $EndComp
 $Comp
@@
 $EndComp
 $Comp
-L 74LS245 U6
-U 1 1 5C81A802
-P 1875 5400
-F 0 "U6" H 1825 5200 60  0000 L BNN
-F 1 "74LS245" H 1675 5450 60  0000 L TNN
-F 2 "~" H 1875 5400 60  0000 C CNN
-F 3 "~" H 1875 5400 60  0000 C CNN
-	1    1875 5400
-	1    0    0    -1
-$EndComp
-$Comp
 L CONN_8 P3
 U 1 1 5C81A843
@@
 Text Label 2450 1550 0    60   ~ 0
 A8
-Text Label 2450 1650 0    60   ~ 0
-A7
-Text Label 2450 1750 0    60   ~ 0
-A6
-Text Label 2450 1850 0    60   ~ 0
-A5
-Text Label 2450 1950 0    60   ~ 0
-A4
-Text Label 2450 2050 0    60   ~ 0
-A3
-Text Label 2450 2150 0    60   ~ 0
-A2
-Text Label 2450 2250 0    60   ~ 0
-A1
 Entry Wire Line
 	2875 1550 2975 1650
@@
 	1    0    0    -1
 $EndComp
-Text Label 1325 3075 0    60   ~ 0
+Text Label 1325 3175 0    60   ~ 0
 Negative?
-Text Label 1325 3175 0    60   ~ 0
+Text Label 1325 3375 0    60   ~ 0
 INC
-Text Label 1325 3275 0    60   ~ 0
+Text Label 1325 3575 0    60   ~ 0
 Sum Out
-Text Label 1325 3375 0    60   ~ 0
+Text Label 1325 3675 0    60   ~ 0
 Subtract
 Text Label 1325 3475 0    60   ~ 0
 Not Zero?
-Text Label 1325 3575 0    60   ~ 0
+Text Label 1325 3275 0    60   ~ 0
 Odd?
-Text Label 1325 3675 0    60   ~ 0
+Text Label 1325 3075 0    60   ~ 0
 Carry?
 $Comp
 L 9-PIN_HEADER JP1
 U 1 1 5C847A3A
-P 2300 3375
-F 0 "JP1" H 2300 3275 60  0000 C CNN
-F 1 "Blinkenlights" H 2300 3375 60  0000 C CNN
-F 2 "" H 2300 3375 60  0000 C CNN
-F 3 "" H 2300 3375 60  0000 C CNN
-	1    2300 3375
-	0    -1   -1   0
+P 2300 4000
+F 0 "JP1" H 2300 3900 60  0000 C CNN
+F 1 "Blinkenlights" H 2300 4000 60  0000 C CNN
+F 2 "" H 2300 4000 60  0000 C CNN
+F 3 "" H 2300 4000 60  0000 C CNN
+	1    2300 4000
+	1    0    0    -1
 $EndComp
 $Comp
 L GND #PWR012
 U 1 1 5C847C07
-P 2050 3925
-F 0 "#PWR012" H 2050 3925 30  0001 C CNN
-F 1 "GND" H 2050 3855 30  0001 C CNN
-F 2 "" H 2050 3925 60  0000 C CNN
-F 3 "" H 2050 3925 60  0000 C CNN
-	1    2050 3925
+P 1575 3850
+F 0 "#PWR012" H 1575 3850 30  0001 C CNN
+F 1 "GND" H 1575 3780 30  0001 C CNN
+F 2 "" H 1575 3850 60  0000 C CNN
+F 3 "" H 1575 3850 60  0000 C CNN
+	1    1575 3850
 	1    0    0    -1
 $EndComp
@@
 Text Label 8325 2700 0    60   ~ 0
 Sum5
-Text Label 8325 2800 0    60   ~ 0
+Text Label 8350 2800 0    60   ~ 0
 Sum4
 Text Label 8325 2900 0    60   ~ 0
 Sum3
-Text Label 8325 3000 0    60   ~ 0
+Text Label 8350 3000 0    60   ~ 0
 Sum2
 Text Label 8325 3100 0    60   ~ 0
@@
 Text Notes 1750 1400 0    60   ~ 0
 Direct link to register A
-Text Notes 550  4550 0    60   ~ 0
+Text Notes 550  4225 0    60   ~ 0
 Direct link to register B
 Text Notes 1200 7250 0    60   ~ 0
@@
 	4675 3300 4550 3300
 Wire Wire Line
-	1050 4900 1275 4900
-Wire Wire Line
-	1050 5000 1275 5000
-Wire Wire Line
-	1050 5100 1275 5100
-Wire Wire Line
-	1050 5200 1275 5200
-Wire Wire Line
-	1050 5300 1275 5300
-Wire Wire Line
-	1050 5400 1275 5400
-Wire Wire Line
-	1050 5500 1275 5500
-Wire Wire Line
-	1050 5600 1275 5600
-Wire Wire Line
-	1275 5850 1150 5850
-Wire Wire Line
-	1150 4650 1150 6950
-Wire Wire Line
-	1150 4650 1875 4650
-Wire Wire Line
-	1325 2975 2050 2975
-Wire Wire Line
-	1325 3075 2050 3075
-Wire Wire Line
-	1325 3175 2050 3175
-Wire Wire Line
-	1325 3275 2050 3275
-Wire Wire Line
-	1325 3375 2050 3375
-Wire Wire Line
-	1325 3475 2050 3475
-Wire Wire Line
-	1325 3575 2050 3575
-Wire Wire Line
-	1325 3675 2050 3675
-Wire Wire Line
-	2050 3775 2050 3925
-Wire Wire Line
-	1150 6950 2475 6950
-Connection ~ 1150 5850
+	1025 5850 1275 5850
+Wire Wire Line
+	1325 3075 2700 3075
+Wire Wire Line
+	1325 3175 2100 3175
+Wire Wire Line
+	1325 3275 2600 3275
+Wire Wire Line
+	1325 3375 2200 3375
+Wire Wire Line
+	1325 3475 2500 3475
+Wire Wire Line
+	1325 3575 2300 3575
+Wire Wire Line
+	1325 3675 2400 3675
 Wire Wire Line
 	3950 6550 3950 6975
@@
 	3350 4150 2900 4150
 Connection ~ 3350 4150
-Wire Wire Line
-	8575 3350 8050 3350
-Wire Wire Line
-	8050 3350 8050 2150
-Wire Wire Line
-	8050 2150 9175 2150
 Wire Wire Line
 	8575 2400 8325 2400
@@
 	3350 4600 3475 4600
 Connection ~ 3350 4800
+Text Label 2450 1650 0    60   ~ 0
+A1
+Text Label 2450 1750 0    60   ~ 0
+A7
+Text Label 2450 1850 0    60   ~ 0
+A2
+Text Label 2450 1950 0    60   ~ 0
+A6
+Text Label 2450 2050 0    60   ~ 0
+A3
+Text Label 2450 2150 0    60   ~ 0
+A5
+Text Label 2450 2250 0    60   ~ 0
+A4
+$Comp
+L 74LS245 U6
+U 1 1 5C81A802
+P 1875 5400
+F 0 "U6" H 1825 5200 60  0000 L BNN
+F 1 "74LS245" H 1675 5450 60  0000 L TNN
+F 2 "~" H 1875 5400 60  0000 C CNN
+F 3 "~" H 1875 5400 60  0000 C CNN
+	1    1875 5400
+	1    0    0    -1
+$EndComp
+Wire Wire Line
+	1275 4750 1275 4900
+Wire Wire Line
+	1175 4750 1175 5600
+Wire Wire Line
+	1175 5600 1275 5600
+Wire Wire Line
+	1075 4750 1075 5000
+Wire Wire Line
+	1075 5000 1275 5000
+Wire Wire Line
+	975  4750 975  5500
+Wire Wire Line
+	975  5500 1275 5500
+Wire Wire Line
+	875  4750 875  5100
+Wire Wire Line
+	875  5100 1275 5100
+Wire Wire Line
+	775  4750 775  5400
+Wire Wire Line
+	775  5400 1275 5400
+Wire Wire Line
+	675  4750 675  5200
+Wire Wire Line
+	675  5200 1275 5200
+Wire Wire Line
+	575  4750 575  5300
+Wire Wire Line
+	575  5300 1275 5300
+$Comp
+L +5V #PWR016
+U 1 1 5E23B821
+P 1025 5850
+F 0 "#PWR016" H 1025 5940 20  0001 C CNN
+F 1 "+5V" H 1025 5940 30  0000 C CNN
+F 2 "" H 1025 5850 60  0000 C CNN
+F 3 "" H 1025 5850 60  0000 C CNN
+	1    1025 5850
+	1    0    0    -1
+$EndComp
+Wire Wire Line
+	1275 5850 1275 6950
+Wire Wire Line
+	1275 6950 2475 6950
+$Comp
+L +5V #PWR017
+U 1 1 5E23BE9C
+P 8500 3350
+F 0 "#PWR017" H 8500 3440 20  0001 C CNN
+F 1 "+5V" H 8500 3440 30  0000 C CNN
+F 2 "" H 8500 3350 60  0000 C CNN
+F 3 "" H 8500 3350 60  0000 C CNN
+	1    8500 3350
+	1    0    0    -1
+$EndComp
+Wire Wire Line
+	8575 3350 8500 3350
+Wire Wire Line
+	1900 3750 1575 3750
+Wire Wire Line
+	1575 3750 1575 3850
+Wire Wire Line
+	2700 3075 2700 3750
+Wire Wire Line
+	2100 3175 2100 3750
+Wire Wire Line
+	2600 3275 2600 3750
+Wire Wire Line
+	2200 3375 2200 3750
+Wire Wire Line
+	2500 3475 2500 3750
+Wire Wire Line
+	2300 3575 2300 3750
+Wire Wire Line
+	2400 3675 2400 3750
+Wire Wire Line
+	2000 3750 2000 2975
+Wire Wire Line
+	2000 2975 1325 2975
 $EndSCHEMATC

Commit message: v1.5.18 upgraded to KiCad 4.0.5
Parts:
- RA1: symbol R-ARRAY-8 -> R-array-8
Changed lines of the file:
@@
 EESchema Schematic File Version 2
+LIBS:Hol-1-ALU-rescue
 LIBS:benningtons
 LIBS:power
@@
 LIBS:memory
 LIBS:xilinx
-LIBS:special
 LIBS:microcontrollers
 LIBS:dsp
@@
 LIBS:valves
 LIBS:Hol-1-ALU-cache
-EELAYER 27 0
+EELAYER 25 0
 EELAYER END
 $Descr A4 11693 8268
@@
 $EndComp
 $Comp
-L R-ARRAY-8 RA1
+L R-array-8 RA1
 U 1 1 5C81D152
 P 3000 6900
@@
 Text Notes 550  4225 0    60   ~ 0
 Direct link to register B
-Text Notes 1200 7250 0    60   ~ 0
+Text Notes 1200 7550 0    60   ~ 0
 INC: Switch off input from B register and replace by 00000001\nusing pull-down resistor array and one pull-up resistor\n\nDEC: achieved by using INC and Subtract commands
 Text Notes 3450 4150 0    60   ~ 0
@@
 Text Notes 8850 6150 0    60   ~ 0
 16-way IDC ribbon cable\nheaders (right) wired in\nvertical pairs, provides a\n4 port Data Bus for Hol-1
-Text Notes 9450 1950 0    60   ~ 0
+Text Notes 9450 2100 0    60   ~ 0
 Note: the status flags resulting from\nany sum can be tested without\nhaving to place the result onto the\nData Bus, using Sum-Out (below)
 Text Notes 6250 1800 0    60   ~ 0

Commit message: v1.5.19 upgraded to KiCad 5.0
Parts:
- C1, C2, C3: symbol C -> Hol-1-ALU-rescue:C
- D1, D2, D3, D4, D5, D6, D7, D8: symbol DIODE -> Hol-1-ALU-rescue:DIODE
- JP1, JP2: symbol 9-PIN_HEADER -> Hol-1-ALU-rescue:9-PIN_HEADER
- P1, P2, P3: symbol CONN_8 -> Hol-1-ALU-rescue:CONN_8
- P4, P5, P6, P7: symbol CONN_8X2 -> Hol-1-ALU-rescue:CONN_8X2
- P8: symbol CONN_2 -> Hol-1-ALU-rescue:CONN_2
- R1: symbol R -> Hol-1-ALU-rescue:R
- RA1: symbol R-array-8 -> Hol-1-ALU-rescue:R-array-8
- U1, U2: symbol 74LS283 -> Hol-1-ALU-rescue:74LS283
- U3, U4: symbol 74LS86 -> Hol-1-ALU-rescue:74LS86
- U5, U6: symbol 74LS245 -> Hol-1-ALU-rescue:74LS245
Other:
- moved on the sheet: P4, P5, P6, P7, U5

Commit message: v1.5.20 corrections to remove KiCad rescue libraries
Parts:
- C1, C2, C3: symbol Hol-1-ALU-rescue:C -> benningtons:C
- D1, D2, D3, D4, D5, D6, D7, D8: symbol Hol-1-ALU-rescue:DIODE -> benningtons:DIODE
- JP1, JP2: symbol Hol-1-ALU-rescue:9-PIN_HEADER -> benningtons:9-PIN_HEADER
- P1, P2, P3: symbol Hol-1-ALU-rescue:CONN_8 -> benningtons:CONN_8
- P4, P5, P6, P7: symbol Hol-1-ALU-rescue:CONN_8X2 -> benningtons:CONN_8X2
- P8: symbol Hol-1-ALU-rescue:CONN_2 -> benningtons:CONN_2
- R1: symbol Hol-1-ALU-rescue:R -> benningtons:R
- RA1: symbol Hol-1-ALU-rescue:R-array-8 -> benningtons:R-array-8
- U1, U2: symbol Hol-1-ALU-rescue:74LS283 -> benningtons:74LS283
- U3, U4: symbol Hol-1-ALU-rescue:74LS86 -> benningtons:74LS86
- U5, U6: symbol Hol-1-ALU-rescue:74LS245 -> benningtons:74LS245
Changed lines of the file:
@@
 EESchema Schematic File Version 4
-LIBS:Hol-1-ALU-cache
-EELAYER 26 0
+EELAYER 30 0
 EELAYER END
 $Descr A4 11693 8268
@@
 $EndDescr
 $Comp
-L Hol-1-ALU-rescue:CONN_8 P2
+L benningtons:CONN_8 P2
 U 1 1 5C5A0CA2
 P 925 4400
@@
 $EndComp
 $Comp
-L Hol-1-ALU-rescue:CONN_8 P1
+L benningtons:CONN_8 P1
 U 1 1 5C5A0CC3
 P 2100 1900
@@
 $EndComp
 $Comp
-L Hol-1-ALU-rescue:PWR_FLAG #FLG01
+L benningtons:PWR_FLAG #FLG01
 U 1 1 5C5E3694
 P 5150 6625
@@
 $EndComp
 $Comp
-L Hol-1-ALU-rescue:PWR_FLAG #FLG02
+L benningtons:PWR_FLAG #FLG02
 U 1 1 5C5E36A1
 P 6625 7325
@@
 $EndComp
 $Comp
-L Hol-1-ALU-rescue:GND #PWR03
+L benningtons:GND #PWR03
 U 1 1 5C5E36D8
 P 6475 7450
@@
 $EndComp
 $Comp
-L Hol-1-ALU-rescue:74LS245 U5
+L benningtons:74LS245 U5
 U 1 1 5C607B53
 P 9175 2500
@@
 $EndComp
 $Comp
-L Hol-1-ALU-rescue:GND #PWR04
+L benningtons:GND #PWR04
 U 1 1 5C607B70
 P 9175 3250
@@
 $EndComp
 $Comp
-L Hol-1-ALU-rescue:9-PIN_HEADER JP2
+L benningtons:9-PIN_HEADER JP2
 U 1 1 5C608CCD
 P 7150 5200
@@
 $EndComp
 $Comp
-L Hol-1-ALU-rescue:C C1
+L benningtons:C C1
 U 1 1 5C60D0BB
 P 6025 6975
@@
 $EndComp
 $Comp
-L Hol-1-ALU-rescue:C C2
+L benningtons:C C2
 U 1 1 5C60D0D2
 P 6250 6975
@@
 $EndComp
 $Comp
-L Hol-1-ALU-rescue:C C3
+L benningtons:C C3
 U 1 1 5C60D0D8
 P 6475 6975
@@
 $EndComp
 $Comp
-L Hol-1-ALU-rescue:+5V #PWR05
+L benningtons:+5V #PWR05
 U 1 1 5C60D23A
 P 5275 6525
@@
 $EndComp
 $Comp
-L Hol-1-ALU-rescue:+5V #PWR06
+L benningtons:+5V #PWR06
 U 1 1 5C60D2F3
 P 9175 1750
@@
 $EndComp
 $Comp
-L Hol-1-ALU-rescue:CONN_2 P8
+L benningtons:CONN_2 P8
 U 1 1 5C71F9E9
 P 4800 7000
@@
 $EndComp
 $Comp
-L Hol-1-ALU-rescue:CONN_8X2 P4
+L benningtons:CONN_8X2 P4
 U 1 1 5C81A7CD
 P 10600 3400
@@
 $EndComp
 $Comp
-L Hol-1-ALU-rescue:CONN_8 P3
+L benningtons:CONN_8 P3
 U 1 1 5C81A843
 P 975 3325
@@
 $EndComp
 $Comp
-L Hol-1-ALU-rescue:74LS283 U1
+L benningtons:74LS283 U1
 U 1 1 5C81AD95
 P 5275 1550
@@
 $EndComp
 $Comp
-L Hol-1-ALU-rescue:74LS283 U2
+L benningtons:74LS283 U2
 U 1 1 5C81ADA2
 P 5275 3450
@@
 $EndComp
 $Comp
-L Hol-1-ALU-rescue:74LS86 U3
+L benningtons:74LS86 U3
 U 3 1 5C81C8AD
 P 3800 4850
@@
 $EndComp
 $Comp
-L Hol-1-ALU-rescue:74LS86 U3
+L benningtons:74LS86 U3
 U 4 1 5C81C8BA
 P 3800 5050
@@
 $EndComp
 $Comp
-L Hol-1-ALU-rescue:74LS86 U3
+L benningtons:74LS86 U3
 U 1 1 5C81C8C2
 P 3800 5250
@@
 $EndComp
 $Comp
-L Hol-1-ALU-rescue:74LS86 U3
+L benningtons:74LS86 U3
 U 2 1 5C81C8D1
 P 3800 5450
@@
 $EndComp
 $Comp
-L Hol-1-ALU-rescue:74LS86 U4
+L benningtons:74LS86 U4
 U 3 1 5C81C8E0
 P 3800 5650
@@
 $EndComp
 $Comp
-L Hol-1-ALU-rescue:74LS86 U4
+L benningtons:74LS86 U4
 U 4 1 5C81C8EF
 P 3800 5850
@@
 $EndComp
 $Comp
-L Hol-1-ALU-rescue:74LS86 U4
+L benningtons:74LS86 U4
 U 1 1 5C81C8FE
 P 3800 6050
@@
 $EndComp
 $Comp
-L Hol-1-ALU-rescue:74LS86 U4
+L benningtons:74LS86 U4
 U 2 1 5C81C90D
 P 3800 6250
@@
 $EndComp
 $Comp
-L Hol-1-ALU-rescue:74LS86 U3
+L benningtons:74LS86 U3
 U 5 1 5C81C91C
 P 5475 6975
@@
 $EndComp
 $Comp
-L Hol-1-ALU-rescue:74LS86 U4
+L benningtons:74LS86 U4
 U 5 1 5C81C938
 P 5775 6975
@@
 $EndComp
 $Comp
-L Hol-1-ALU-rescue:DIODE D7
+L benningtons:DIODE D7
 U 1 1 5C81CBC0
 P 7975 4650
@@
 $EndComp
 $Comp
-L Hol-1-ALU-rescue:DIODE D6
+L benningtons:DIODE D6
 U 1 1 5C81CC4B
 P 7975 4500
@@
 $EndComp
 $Comp
-L Hol-1-ALU-rescue:DIODE D5
+L benningtons:DIODE D5
 U 1 1 5C81CC5A
 P 7975 4350
@@
 $EndComp
 $Comp
-L Hol-1-ALU-rescue:DIODE D1
+L benningtons:DIODE D1
 U 1 1 5C81CC69
 P 7975 3750
@@
 $EndComp
 $Comp
-L Hol-1-ALU-rescue:DIODE D8
+L benningtons:DIODE D8
 U 1 1 5C81CC78
 P 7975 4800
@@
 $EndComp
 $Comp
-L Hol-1-ALU-rescue:DIODE D4
+L benningtons:DIODE D4
 U 1 1 5C81CC87
 P 7975 4200
@@
 $EndComp
 $Comp
-L Hol-1-ALU-rescue:DIODE D3
+L benningtons:DIODE D3
 U 1 1 5C81CC96
 P 7975 4050
@@
 $EndComp
 $Comp
-L Hol-1-ALU-rescue:DIODE D2
+L benningtons:DIODE D2
 U 1 1 5C81CCA5
 P 7975 3900
@@
 $EndComp
 $Comp
-L Hol-1-ALU-rescue:R-array-8 RA1
+L benningtons:R-array-8 RA1
 U 1 1 5C81D152
 P 3000 6900
@@
 $EndComp
 $Comp
-L Hol-1-ALU-rescue:R R1
+L benningtons:R R1
 U 1 1 5C81D24A
 P 2475 6750
@@
 A8
 $Comp
-L Hol-1-ALU-rescue:+5V #PWR07
+L benningtons:+5V #PWR07
 U 1 1 5C8474A4
 P 5275 800
@@
 $EndComp
 $Comp
-L Hol-1-ALU-rescue:+5V #PWR08
+L benningtons:+5V #PWR08
 U 1 1 5C8474AA
 P 5275 2700
@@
 $EndComp
 $Comp
-L Hol-1-ALU-rescue:+5V #PWR09
+L benningtons:+5V #PWR09
 U 1 1 5C8474B0
 P 1875 4650
@@
 $EndComp
 $Comp
-L Hol-1-ALU-rescue:GND #PWR010
+L benningtons:GND #PWR010
 U 1 1 5C847526
 P 5275 4200
@@
 $EndComp
 $Comp
-L Hol-1-ALU-rescue:GND #PWR011
+L benningtons:GND #PWR011
 U 1 1 5C84752C
 P 5275 2300
@@
 Carry?
 $Comp
-L Hol-1-ALU-rescue:9-PIN_HEADER JP1
+L benningtons:9-PIN_HEADER JP1
 U 1 1 5C847A3A
 P 2300 4000
@@
 $EndComp
 $Comp
-L Hol-1-ALU-rescue:GND #PWR012
+L benningtons:GND #PWR012
 U 1 1 5C847C07
 P 1575 3850
@@
 INC
 $Comp
-L Hol-1-ALU-rescue:GND #PWR013
+L benningtons:GND #PWR013
 U 1 1 5C847520
 P 1875 6150
@@
 $EndComp
 $Comp
-L Hol-1-ALU-rescue:GND #PWR014
+L benningtons:GND #PWR014
 U 1 1 5C850142
 P 3950 6975
@@
 Negative?
 $Comp
-L Hol-1-ALU-rescue:GND #PWR015
+L benningtons:GND #PWR015
 U 1 1 5C855E86
 P 7825 5225
@@
 $EndComp
 $Comp
-L Hol-1-ALU-rescue:CONN_8X2 P5
+L benningtons:CONN_8X2 P5
 U 1 1 5C856897
 P 10600 4300
@@
 $EndComp
 $Comp
-L Hol-1-ALU-rescue:CONN_8X2 P6
+L benningtons:CONN_8X2 P6
 U 1 1 5C85689D
 P 10600 5200
@@
 $EndComp
 $Comp
-L Hol-1-ALU-rescue:CONN_8X2 P7
+L benningtons:CONN_8X2 P7
 U 1 1 5C8568A3
 P 10600 6100
@@
 A4
 $Comp
-L Hol-1-ALU-rescue:74LS245 U6
+L benningtons:74LS245 U6
 U 1 1 5C81A802
 P 1875 5400
@@
 	575  5300 1275 5300
 $Comp
-L Hol-1-ALU-rescue:+5V #PWR016
+L benningtons:+5V #PWR016
 U 1 1 5E23B821
 P 1025 5850
@@
 	1275 6950 2475 6950
 $Comp
-L Hol-1-ALU-rescue:+5V #PWR017
+L benningtons:+5V #PWR017
 U 1 1 5E23BE9C
 P 8500 2950
@@
 Wire Wire Line
 	10950 2300 10950 3000
+Connection ~ 10950 3000
 Wire Bus Line
 	4450 1000 4450 1300
@@
 Wire Bus Line
 	2975 1000 2975 1950
-Connection ~ 10950 3000
 $EndSCHEMATC
