File: MMU/Hol-1-MMU.sch (KiCad schematic (older format))
At the start: 36 parts, among them P1 DATA BUS, P2 ADDRESS PORT, P3 DATA PORT, P4 MMU CONTROL, P5 Power, SW1 HEX_SWITCH, SW2 HEX_SWITCH, SW3 HEX_SWITCH, SW4 HEX_SWITCH, SW5 DPDT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

Commit message: v1.5.16 MMU: don't share a resistor between program and run LEDs
Parts:
- added R3: 220Ω, ~, symbol R
Other:
- moved on the sheet: R1
Changed lines of the file:
@@
 Sheet 1 1
 Title "Hol-1 8-bit CPU - Memory Management Unit"
-Date "8 sep 2019"
+Date "29 jan 2020"
 Rev "1"
 Comp "www.benningtons.net"
@@
 L R R1
 U 1 1 5D0FDFE4
-P 10600 2550
-F 0 "R1" V 10725 2550 40  0000 C CNN
-F 1 "220Ω" V 10500 2550 40  0000 C CNN
-F 2 "~" V 10530 2550 30  0000 C CNN
-F 3 "~" H 10600 2500 30  0000 C CNN
-	1    10600 2550
+P 10700 2550
+F 0 "R1" V 10800 2450 40  0000 C CNN
+F 1 "220Ω" V 10800 2600 40  0000 C CNN
+F 2 "~" V 10630 2550 30  0000 C CNN
+F 3 "~" H 10700 2500 30  0000 C CNN
+	1    10700 2550
 	1    0    0    -1
 $EndComp
@@
 Note: Rotary switches (SW1-4)\nselect 0 to F and output the\nresult in 4-bits.
 $Comp
-L DPDT SW5
-U 1 1 5D2B21C4
-P 10600 3850
-F 0 "SW5" H 10400 4000 50  0000 C CNN
-F 1 "DPDT" H 10450 3700 50  0001 C CNN
-F 2 "~" H 10600 3850 60  0000 C CNN
-F 3 "~" H 10600 3850 60  0000 C CNN
-	1    10600 3850
-	0    -1   -1   0
-$EndComp
-$Comp
 L CONN_2 P5
 U 1 1 5D3C5DD9
@@
 	10700 2750 10700 2850
 Wire Wire Line
-	10500 2750 10700 2750
-Connection ~ 10600 2750
-Wire Wire Line
 	3400 1700 3500 1700
 Connection ~ 3500 1700
@@
 	9600 6750 9500 6750
 Connection ~ 9500 6750
+$Comp
+L DPDT SW5
+U 1 1 5D8007A6
+P 10600 3850
+F 0 "SW5" H 10400 4000 50  0000 C CNN
+F 1 "DPDT" H 10450 3700 50  0001 C CNN
+F 2 "~" H 10600 3850 60  0000 C CNN
+F 3 "~" H 10600 3850 60  0000 C CNN
+	1    10600 3850
+	0    -1   -1   0
+$EndComp
+$Comp
+L R R3
+U 1 1 5E31EEDA
+P 10500 2550
+F 0 "R3" V 10400 2450 40  0000 C CNN
+F 1 "220Ω" V 10400 2600 40  0000 C CNN
+F 2 "~" V 10430 2550 30  0000 C CNN
+F 3 "~" H 10500 2500 30  0000 C CNN
+	1    10500 2550
+	1    0    0    -1
+$EndComp
+Wire Wire Line
+	10500 2350 10700 2350
+Connection ~ 10600 2350
 $EndSCHEMATC

Commit message: v1.5.18 upgraded to KiCad 4.0.5
Parts:
- RA1, RA2: symbol R-ARRAY-8 -> R-array-8
Changed lines of the file:
@@
 EESchema Schematic File Version 2
+LIBS:Hol-1-MMU-rescue
 LIBS:benningtons
 LIBS:power
@@
 LIBS:memory
 LIBS:xilinx
-LIBS:special
 LIBS:microcontrollers
 LIBS:dsp
@@
 LIBS:valves
 LIBS:Hol-1-MMU-cache
-EELAYER 27 0
+EELAYER 25 0
 EELAYER END
 $Descr A4 11693 8268
@@
 $EndComp
 $Comp
-L R-ARRAY-8 RA1
+L R-array-8 RA1
 U 1 1 5D0EBE15
 P 6450 4450
@@
 $EndComp
 $Comp
-L R-ARRAY-8 RA2
+L R-array-8 RA2
 U 1 1 5D1005E6
 P 3450 7650

Commit message: v1.5.19 upgraded to KiCad 5.0
Parts:
- C1, C2, C3, C4, C5, C6, C7, C8: symbol C -> Hol-1-MMU-rescue:C
- D1, D2: symbol LED -> Hol-1-MMU-rescue:LED
- JP1, JP2: symbol 10-PIN_HEADER -> Hol-1-MMU-rescue:10-PIN_HEADER
- JP3: symbol 9-PIN_HEADER -> Hol-1-MMU-rescue:9-PIN_HEADER
- P1: symbol CONN_8X2 -> Hol-1-MMU-rescue:CONN_8X2
- P2, P3, P4: symbol CONN_8 -> Hol-1-MMU-rescue:CONN_8
- P5: symbol CONN_2 -> Hol-1-MMU-rescue:CONN_2
- R1, R2, R3: symbol R -> Hol-1-MMU-rescue:R
- RA1, RA2: symbol R-array-8 -> Hol-1-MMU-rescue:R-array-8
- SW1, SW2, SW3, SW4: symbol CODE_SWITCH -> Hol-1-MMU-rescue:CODE_SWITCH
- SW5: symbol DPDT -> Hol-1-MMU-rescue:DPDT
- SW6: symbol SW_PUSH -> Hol-1-MMU-rescue:SW_PUSH
- U1: symbol 74LS00 -> Hol-1-MMU-rescue:74LS00
- U2, U4: symbol 74LS173 -> Hol-1-MMU-rescue:74LS173
- U3, U5, U6, U7, U8: symbol 74LS157 -> Hol-1-MMU-rescue:74LS157
Connections:
- wire segments 232 -> 316
Other:
- moved on the sheet: C1, P4, R2, SW6, U1A, U7

Commit message: v1.5.20 corrections to remove KiCad rescue libraries
Parts:
- C1, C2, C3, C4, C5, C6, C7, C8: symbol Hol-1-MMU-rescue:C -> benningtons:C
- D1, D2: symbol Hol-1-MMU-rescue:LED -> benningtons:LED
- JP1, JP2: symbol Hol-1-MMU-rescue:10-PIN_HEADER -> benningtons:10-PIN_HEADER
- JP3: symbol Hol-1-MMU-rescue:9-PIN_HEADER -> benningtons:9-PIN_HEADER
- P1: symbol Hol-1-MMU-rescue:CONN_8X2 -> benningtons:CONN_8X2
- P2, P3, P4: symbol Hol-1-MMU-rescue:CONN_8 -> benningtons:CONN_8
- P5: symbol Hol-1-MMU-rescue:CONN_2 -> benningtons:CONN_2
- R1, R2, R3: symbol Hol-1-MMU-rescue:R -> benningtons:R
- RA1, RA2: symbol Hol-1-MMU-rescue:R-array-8 -> benningtons:R-array-8
- SW1, SW2, SW3, SW4: symbol Hol-1-MMU-rescue:CODE_SWITCH -> benningtons:CODE_SWITCH
- SW5: symbol Hol-1-MMU-rescue:DPDT -> benningtons:DPDT
- SW6: symbol Hol-1-MMU-rescue:SW_PUSH -> benningtons:SW_PUSH
- U1: symbol Hol-1-MMU-rescue:74LS00 -> benningtons:74LS00
- U2, U4: symbol Hol-1-MMU-rescue:74LS173 -> benningtons:74LS173
- U3, U5, U6, U7, U8: symbol Hol-1-MMU-rescue:74LS157 -> benningtons:74LS157
